File: h-ALO-kicad-libs.kicad_sch (KiCad schematic)
At the start: 0 parts

Commit message: update
Parts:
- added J1: 6P6C, Connector_RJ:RJ25_Wayconn_MJEA-660X1_Horizontal, symbol Connector:6P6C
- added U1: h-ALO-sensor, h-ALO:h-ALO-sensor, symbol h-ALO:h-ALO-sensor
Connections:
- new net: J1.6, U1.1 (OPD1)
- new net: J1.4, U1.2 (OPD2)
- new net: J1.2, U1.3 (OPD3)
Changed lines of the file:
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@@
 (kicad_sch (version 20211123) (generator eeschema)
   (paper "A4")
-  (symbol_instances)
+  (wire (pts (xy 87.63 81.28) (xy 119.38 81.28))
+    (stroke (width 0) (type default) (color 0 0 0 0))
+  )
+  (wire (pts (xy 93.98 77.47) (xy 93.98 76.2))
+    (stroke (width 0) (type default) (color 0 0 0 0))
+  )
+  (wire (pts (xy 119.38 77.47) (xy 93.98 77.47))
+    (stroke (width 0) (type default) (color 0 0 0 0))
+  )
+  (wire (pts (xy 87.63 71.12) (xy 119.38 71.12))
+    (stroke (width 0) (type default) (color 0 0 0 0))
+  )
+  (wire (pts (xy 93.98 76.2) (xy 87.63 76.2))
+    (stroke (width 0) (type default) (color 0 0 0 0))
+  )
+  (wire (pts (xy 119.38 71.12) (xy 119.38 73.66))
+    (stroke (width 0) (type default) (color 0 0 0 0))
+  )
+  (symbol (lib_id "h-ALO:h-ALO-sensor") (at 134.62 83.82 0) (unit 1)
+    (in_bom yes) (on_board yes) (fields_autoplaced)
+    (property "Reference" "U1" (id 0) (at 163.83 80.0099 0)
+      (effects (font (size 1.27 1.27)) (justify left))
+    )
+    (property "Value" "h-ALO-sensor" (id 1) (at 163.83 82.5499 0)
+      (effects (font (size 1.27 1.27)) (justify left))
+    )
+    (property "Footprint" "h-ALO:h-ALO-sensor" (id 2) (at 140.97 72.39 0)
+      (effects (font (size 1.27 1.27)) hide)
+    )
+    (property "Datasheet" "" (id 3) (at 134.62 83.82 0)
+      (effects (font (size 1.27 1.27)) hide)
+    )
+    (pin "1")
+    (pin "2")
+    (pin "3")
+  )
+  (symbol (lib_id "Connector:6P6C") (at 77.47 78.74 0) (unit 1)
+    (in_bom yes) (on_board yes) (fields_autoplaced)
+    (property "Reference" "J1" (id 0) (at 77.47 63.5 0))
+    (property "Value" "6P6C" (id 1) (at 77.47 66.04 0))
+    (property "Footprint" "Connector_RJ:RJ25_Wayconn_MJEA-660X1_Horizontal" (id 2) (at 77.47 78.105 90)
+      (effects (font (size 1.27 1.27)) hide)
+    )
+    (property "Datasheet" "~" (id 3) (at 77.47 78.105 90)
+      (effects (font (size 1.27 1.27)) hide)
+    )
+    (pin "1")
+    (pin "2")
+    (pin "3")
+    (pin "4")
+    (pin "5")
+    (pin "6")
+  )
+  (sheet_instances
+    (path "/" (page "1"))
+  )
+  (symbol_instances
+    (path "/ad8cdddf-61ae-43a2-ac2b-d061f53a3281"
+      (reference "J1") (unit 1) (value "6P6C") (footprint "Connector_RJ:RJ25_Wayconn_MJEA-660X1_Horizontal")
+    )
+    (path "/3e52c28f-3453-4672-a557-9f75bfe95a96"
+      (reference "U1") (unit 1) (value "h-ALO-sensor") (footprint "h-ALO:h-ALO-sensor")
+    )
+  )
 )

Commit message: update
Parts:
- added U2: LOG114AIRGVR, Package_DFN_QFN:QFN-16-1EP_4x4mm_P0.65mm_EP2.15x2.15mm, symbol LOG114:LOG114AIRGVR
Connections:
- net at J1.4, U1.2 (OPD2): now also U2.16 (VREF)
- net at J1.2, U1.3 (OPD3): now also U2.13 (+IN5)
Changed lines of the file:
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@@
 (kicad_sch (version 20211123) (generator eeschema)
   (paper "A4")
-  (wire (pts (xy 87.63 81.28) (xy 119.38 81.28))
+  (junction (at 101.6 81.28) (diameter 0) (color 0 0 0 0)
+  )
+  (junction (at 93.98 77.47) (diameter 0) (color 0 0 0 0)
+  )
+  (wire (pts (xy 87.63 81.28) (xy 101.6 81.28))
     (stroke (width 0) (type default) (color 0 0 0 0))
   )
@@
   )
   (wire (pts (xy 119.38 77.47) (xy 93.98 77.47))
+    (stroke (width 0) (type default) (color 0 0 0 0))
+  )
+  (wire (pts (xy 101.6 81.28) (xy 101.6 101.6))
+    (stroke (width 0) (type default) (color 0 0 0 0))
+  )
+  (wire (pts (xy 101.6 81.28) (xy 119.38 81.28))
+    (stroke (width 0) (type default) (color 0 0 0 0))
+  )
+  (wire (pts (xy 93.98 77.47) (xy 93.98 101.6))
     (stroke (width 0) (type default) (color 0 0 0 0))
   )
@@
     (pin "3")
   )
+  (symbol (lib_id "LOG114:LOG114AIRGVR") (at 97.79 118.11 0) (unit 1)
+    (in_bom yes) (on_board yes) (fields_autoplaced)
+    (property "Reference" "U2" (id 0) (at 121.92 108.9912 0))
+    (property "Value" "LOG114AIRGVR" (id 1) (at 121.92 111.5312 0))
+    (property "Footprint" "Package_DFN_QFN:QFN-16-1EP_4x4mm_P0.65mm_EP2.15x2.15mm" (id 2) (at 101.6 92.71 0)
+      (effects (font (size 1.27 1.27)) hide)
+    )
+    (property "Datasheet" "" (id 3) (at 99.06 99.06 0)
+      (effects (font (size 1.27 1.27)) hide)
+    )
+    (pin "")
+    (pin "10")
+    (pin "11")
+    (pin "12")
+    (pin "13")
+    (pin "14")
+    (pin "15")
+    (pin "16")
+    (pin "2")
+    (pin "3")
+    (pin "4")
+    (pin "5")
+    (pin "6")
+    (pin "7")
+    (pin "8")
+    (pin "9")
+  )
   (symbol (lib_id "Connector:6P6C") (at 77.47 78.74 0) (unit 1)
     (in_bom yes) (on_board yes) (fields_autoplaced)
@@
       (reference "U1") (unit 1) (value "h-ALO-sensor") (footprint "h-ALO:h-ALO-sensor")
     )
+    (path "/40c48534-3553-4718-8236-458a9e91dfa5"
+      (reference "U2") (unit 1) (value "LOG114AIRGVR") (footprint "Package_DFN_QFN:QFN-16-1EP_4x4mm_P0.65mm_EP2.15x2.15mm")
+    )
   )

Commit message: Updated h-ALO footprint
Parts:
- removed J1: 6P6C, Connector_RJ:RJ25_Wayconn_MJEA-660X1_Horizontal, symbol Connector:6P6C
Connections:
- net at U1.2 (NC): no longer U2.16 (VREF)
- net at U1.3 (Temp): no longer U2.13 (+IN5)
Other:
- moved on the sheet: U2
Changed lines of the file:
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@@
 (kicad_sch (version 20211123) (generator eeschema)
   (paper "A4")
-  (junction (at 101.6 81.28) (diameter 0) (color 0 0 0 0)
-  )
-  (junction (at 93.98 77.47) (diameter 0) (color 0 0 0 0)
-  )
-  (wire (pts (xy 87.63 81.28) (xy 101.6 81.28))
-    (stroke (width 0) (type default) (color 0 0 0 0))
-  )
-  (wire (pts (xy 93.98 77.47) (xy 93.98 76.2))
-    (stroke (width 0) (type default) (color 0 0 0 0))
-  )
-  (wire (pts (xy 119.38 77.47) (xy 93.98 77.47))
-    (stroke (width 0) (type default) (color 0 0 0 0))
-  )
-  (wire (pts (xy 101.6 81.28) (xy 101.6 101.6))
-    (stroke (width 0) (type default) (color 0 0 0 0))
-  )
-  (wire (pts (xy 101.6 81.28) (xy 119.38 81.28))
-    (stroke (width 0) (type default) (color 0 0 0 0))
-  )
-  (wire (pts (xy 93.98 77.47) (xy 93.98 101.6))
-    (stroke (width 0) (type default) (color 0 0 0 0))
-  )
-  (wire (pts (xy 87.63 71.12) (xy 119.38 71.12))
-    (stroke (width 0) (type default) (color 0 0 0 0))
-  )
-  (wire (pts (xy 93.98 76.2) (xy 87.63 76.2))
-    (stroke (width 0) (type default) (color 0 0 0 0))
-  )
-  (wire (pts (xy 119.38 71.12) (xy 119.38 73.66))
-    (stroke (width 0) (type default) (color 0 0 0 0))
-  )
   (symbol (lib_id "h-ALO:h-ALO-sensor") (at 134.62 83.82 0) (unit 1)
-    (in_bom yes) (on_board yes) (fields_autoplaced)
-    (property "Reference" "U1" (id 0) (at 163.83 80.0099 0)
+    (in_bom yes) (on_board yes)
+    (property "Reference" "U1" (id 0) (at 133.35 76.2 0)
       (effects (font (size 1.27 1.27)) (justify left))
     )
-    (property "Value" "h-ALO-sensor" (id 1) (at 163.83 82.5499 0)
+    (property "Value" "h-ALO-sensor" (id 1) (at 132.08 83.82 0)
       (effects (font (size 1.27 1.27)) (justify left))
     )
@@
       (effects (font (size 1.27 1.27)) hide)
     )
+    (pin "10")
+    (pin "11")
+    (pin "12")
+    (pin "13")
+    (pin "14")
+    (pin "15")
+    (pin "16")
+    (pin "17")
+    (pin "18")
+    (pin "19")
+    (pin "2")
+    (pin "20")
+    (pin "21")
+    (pin "22")
+    (pin "23")
+    (pin "24")
+    (pin "25")
+    (pin "26")
+    (pin "27")
+    (pin "28")
+    (pin "3")
+    (pin "30")
+    (pin "31")
+    (pin "32")
+    (pin "33")
+    (pin "34")
+    (pin "35")
+    (pin "36")
+    (pin "37")
+    (pin "38")
+    (pin "39")
+    (pin "4")
+    (pin "40")
+    (pin "41")
+    (pin "42")
+    (pin "43")
+    (pin "44")
+    (pin "45")
+    (pin "46")
+    (pin "47")
+    (pin "48")
+    (pin "49")
+    (pin "5")
+    (pin "50")
+    (pin "51")
+    (pin "52")
+    (pin "53")
+    (pin "54")
+    (pin "55")
+    (pin "56")
+    (pin "6")
+    (pin "7")
+    (pin "8")
+    (pin "9")
     (pin "1")
-    (pin "2")
-    (pin "3")
+    (pin "29")
   )
-  (symbol (lib_id "Connector:6P6C") (at 77.47 78.74 0) (unit 1)
+  (symbol (lib_id "LOG114:LOG114AIRGVR") (at 76.2 115.57 0) (unit 1)
     (in_bom yes) (on_board yes) (fields_autoplaced)
-    (property "Reference" "J1" (id 0) (at 77.47 63.5 0))
-    (property "Value" "6P6C" (id 1) (at 77.47 66.04 0))
-    (property "Footprint" "Connector_RJ:RJ25_Wayconn_MJEA-660X1_Horizontal" (id 2) (at 77.47 78.105 90)
+    (property "Reference" "U2" (id 0) (at 100.33 106.4512 0))
+    (property "Value" "LOG114AIRGVR" (id 1) (at 100.33 108.9912 0))
+    (property "Footprint" "Package_DFN_QFN:QFN-16-1EP_4x4mm_P0.65mm_EP2.15x2.15mm" (id 2) (at 80.01 90.17 0)
       (effects (font (size 1.27 1.27)) hide)
     )
-    (property "Datasheet" "~" (id 3) (at 77.47 78.105 90)
-      (effects (font (size 1.27 1.27)) hide)
-    )
-    (pin "1")
-    (pin "2")
-    (pin "3")
-    (pin "4")
-    (pin "5")
-    (pin "6")
-  )
-  (symbol (lib_id "LOG114:LOG114AIRGVR") (at 97.79 118.11 0) (unit 1)
-    (in_bom yes) (on_board yes) (fields_autoplaced)
-    (property "Reference" "U2" (id 0) (at 121.92 108.9912 0))
-    (property "Value" "LOG114AIRGVR" (id 1) (at 121.92 111.5312 0))
-    (property "Footprint" "Package_DFN_QFN:QFN-16-1EP_4x4mm_P0.65mm_EP2.15x2.15mm" (id 2) (at 101.6 92.71 0)
-      (effects (font (size 1.27 1.27)) hide)
-    )
-    (property "Datasheet" "https://www.ti.com/product/LOG114" (id 3) (at 99.06 99.06 0)
+    (property "Datasheet" "https://www.ti.com/product/LOG114" (id 3) (at 77.47 96.52 0)
       (effects (font (size 1.27 1.27)) hide)
     )
@@
   )
   (symbol_instances
-    (path "/ad8cdddf-61ae-43a2-ac2b-d061f53a3281"
-      (reference "J1") (unit 1) (value "6P6C") (footprint "Connector_RJ:RJ25_Wayconn_MJEA-660X1_Horizontal")
-    )
     (path "/3e52c28f-3453-4672-a557-9f75bfe95a96"
       (reference "U1") (unit 1) (value "h-ALO-sensor") (footprint "h-ALO:h-ALO-sensor")

Commit message: update
Parts:
- added IC1: REF102, Voltage Reference:SO08, symbol Voltage Reference:REF102
Changed lines of the file:
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@@
     (pin "29")
+  )
+  (symbol (lib_id "Voltage Reference:REF102") (at 74.93 55.88 0) (unit 1)
+    (in_bom yes) (on_board yes) (fields_autoplaced)
+    (property "Reference" "IC1" (id 0) (at 74.93 40.64 0))
+    (property "Value" "REF102" (id 1) (at 74.93 43.18 0))
+    (property "Footprint" "Voltage Reference:SO08" (id 2) (at 74.93 55.88 0)
+      (effects (font (size 1.27 1.27)) hide)
+    )
+    (property "Datasheet" "" (id 3) (at 74.93 55.88 0)
+      (effects (font (size 1.27 1.27)) (justify left bottom) hide)
+    )
+    (property "OC_NEWARK" "04M4600" (id 4) (at 74.93 55.88 0)
+      (effects (font (size 1.27 1.27)) (justify left bottom) hide)
+    )
+    (property "MF" "TEXAS INSTRUMENTS" (id 5) (at 74.93 55.88 0)
+      (effects (font (size 1.27 1.27)) (justify left bottom) hide)
+    )
+    (property "MPN" "REF102AU" (id 6) (at 74.93 55.88 0)
+      (effects (font (size 1.27 1.27)) (justify left bottom) hide)
+    )
+    (property "OC_FARNELL" "1212344" (id 7) (at 74.93 55.88 0)
+      (effects (font (size 1.27 1.27)) (justify left bottom) hide)
+    )
+    (pin "1")
+    (pin "2")
+    (pin "3")
+    (pin "4")
+    (pin "5")
+    (pin "6")
+    (pin "7")
+    (pin "8")
   )
   (symbol (lib_id "LOG114:LOG114AIRGVR") (at 76.2 115.57 0) (unit 1)
@@
   )
   (symbol_instances
+    (path "/59834e42-0d61-4573-9fa5-e0d2ae1e3d7c"
+      (reference "IC1") (unit 1) (value "REF102") (footprint "Voltage Reference:SO08")
+    )
     (path "/3e52c28f-3453-4672-a557-9f75bfe95a96"
       (reference "U1") (unit 1) (value "h-ALO-sensor") (footprint "h-ALO:h-ALO-sensor")

Commit message: update
Parts:
- removed IC1: REF102, Voltage Reference:SO08, symbol Voltage Reference:REF102
- added U3: OPA277UA, Package_SO:SOIC-8_3.9x4.9mm_P1.27mm, symbol OPAx277:OPA277UA
- added U4: REF102BU, Package_SO:SOIC-8_3.9x4.9mm_P1.27mm, symbol Reference_Voltage:REF102BU
Changed lines of the file:
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@@
 (kicad_sch (version 20211123) (generator eeschema)
   (paper "A4")
+  (symbol (lib_id "OPAx277:OPA277UA") (at 116.84 39.37 0) (unit 1)
+    (in_bom yes) (on_board yes) (fields_autoplaced)
+    (property "Reference" "U3" (id 0) (at 118.11 20.32 0))
+    (property "Value" "OPA277UA" (id 1) (at 118.11 22.86 0))
+    (property "Footprint" "Package_SO:SOIC-8_3.9x4.9mm_P1.27mm" (id 2) (at 106.68 12.7 0)
+      (effects (font (size 1.27 1.27)) (justify left bottom) hide)
+    )
+    (property "Datasheet" "" (id 3) (at 116.84 39.37 0)
+      (effects (font (size 1.27 1.27)) (justify left bottom) hide)
+    )
+    (property "PARTREV" "02/2019" (id 4) (at 111.76 20.32 0)
+      (effects (font (size 1.27 1.27)) (justify left bottom) hide)
+    )
+    (property "MAXIMUM_PACKAGE_HEIGHT" "1.75 mm" (id 5) (at 111.76 15.24 0)
+      (effects (font (size 1.27 1.27)) (justify left bottom) hide)
+    )
+    (property "STANDARD" "IPC 7351B" (id 6) (at 111.76 17.78 0)
+      (effects (font (size 1.27 1.27)) (justify left bottom) hide)
+    )
+    (property "MANUFACTURER" "Texas Instruments" (id 7) (at 110.49 22.86 0)
+      (effects (font (size 1.27 1.27)) (justify left bottom) hide)
+    )
+    (pin "1")
+    (pin "2")
+    (pin "3")
+    (pin "4")
+    (pin "5")
+    (pin "6")
+    (pin "7")
+    (pin "8")
+  )
   (symbol (lib_id "h-ALO:h-ALO-sensor") (at 134.62 83.82 0) (unit 1)
     (in_bom yes) (on_board yes)
@@
     (pin "29")
   )
-  (symbol (lib_id "Voltage Reference:REF102") (at 74.93 55.88 0) (unit 1)
+  (symbol (lib_id "Reference_Voltage:REF102BU") (at 82.55 80.01 0) (unit 1)
     (in_bom yes) (on_board yes) (fields_autoplaced)
-    (property "Reference" "IC1" (id 0) (at 74.93 40.64 0))
-    (property "Value" "REF102" (id 1) (at 74.93 43.18 0))
-    (property "Footprint" "Voltage Reference:SO08" (id 2) (at 74.93 55.88 0)
-      (effects (font (size 1.27 1.27)) hide)
+    (property "Reference" "U4" (id 0) (at 82.0294 69.85 0)
+      (effects (font (size 1.27 1.27)) (justify left))
     )
-    (property "Datasheet" "" (id 3) (at 74.93 55.88 0)
-      (effects (font (size 1.27 1.27)) (justify left bottom) hide)
+    (property "Value" "REF102BU" (id 1) (at 82.0294 72.39 0)
+      (effects (font (size 1.27 1.27)) (justify left))
     )
-    (property "OC_NEWARK" "04M4600" (id 4) (at 74.93 55.88 0)
-      (effects (font (size 1.27 1.27)) (justify left bottom) hide)
+    (property "Footprint" "Package_SO:SOIC-8_3.9x4.9mm_P1.27mm" (id 2) (at 83.185 86.36 0)
+      (effects (font (size 1.27 1.27) italic) (justify left) hide)
     )
-    (property "MF" "TEXAS INSTRUMENTS" (id 5) (at 74.93 55.88 0)
-      (effects (font (size 1.27 1.27)) (justify left bottom) hide)
-    )
-    (property "MPN" "REF102AU" (id 6) (at 74.93 55.88 0)
-      (effects (font (size 1.27 1.27)) (justify left bottom) hide)
-    )
-    (property "OC_FARNELL" "1212344" (id 7) (at 74.93 55.88 0)
-      (effects (font (size 1.27 1.27)) (justify left bottom) hide)
+    (property "Datasheet" "http://www.ti.com/lit/ds/symlink/ref02.pdf" (id 3) (at 82.55 80.01 0)
+      (effects (font (size 1.27 1.27) italic) hide)
     )
     (pin "1")
@@
   )
   (symbol_instances
-    (path "/59834e42-0d61-4573-9fa5-e0d2ae1e3d7c"
-      (reference "IC1") (unit 1) (value "REF102") (footprint "Voltage Reference:SO08")
-    )
     (path "/3e52c28f-3453-4672-a557-9f75bfe95a96"
       (reference "U1") (unit 1) (value "h-ALO-sensor") (footprint "h-ALO:h-ALO-sensor")
@@
       (reference "U2") (unit 1) (value "LOG114AIRGVR") (footprint "Package_DFN_QFN:QFN-16-1EP_4x4mm_P0.65mm_EP2.15x2.15mm")
     )
+    (path "/3b6a9671-8aa2-4e84-a43a-b66fa7eff663"
+      (reference "U3") (unit 1) (value "OPA277UA") (footprint "Package_SO:SOIC-8_3.9x4.9mm_P1.27mm")
+    )
+    (path "/cb54aeb6-9de6-4b97-aad3-ce0de3c84620"
+      (reference "U4") (unit 1) (value "REF102BU") (footprint "Package_SO:SOIC-8_3.9x4.9mm_P1.27mm")
+    )
   )

Commit message: update
Connections:
- net at U2.10 (+IN4): now also U2.9 (VLOGOUT)
Changed lines of the file:
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@@
 (kicad_sch (version 20211123) (generator eeschema)
   (paper "A4")
+  (wire (pts (xy 71.12 96.52) (xy 71.12 92.71))
+    (stroke (width 0) (type default) (color 0 0 0 0))
+  )
+  (wire (pts (xy 66.04 92.71) (xy 66.04 96.52))
+    (stroke (width 0) (type default) (color 0 0 0 0))
+  )
+  (wire (pts (xy 71.12 92.71) (xy 66.04 92.71))
+    (stroke (width 0) (type default) (color 0 0 0 0))
+  )
   (symbol (lib_id "OPAx277:OPA277UA") (at 116.84 39.37 0) (unit 1)
     (in_bom yes) (on_board yes) (fields_autoplaced)
@@
     (pin "8")
   )
-  (symbol (lib_id "LOG114:LOG114AIRGVR") (at 76.2 115.57 0) (unit 1)
-    (in_bom yes) (on_board yes) (fields_autoplaced)
-    (property "Reference" "U2" (id 0) (at 100.33 106.4512 0))
-    (property "Value" "LOG114AIRGVR" (id 1) (at 100.33 108.9912 0))
-    (property "Footprint" "Package_DFN_QFN:QFN-16-1EP_4x4mm_P0.65mm_EP2.15x2.15mm" (id 2) (at 80.01 90.17 0)
+  (symbol (lib_id "LOG114:LOG114AIRGVR") (at 60.96 118.11 0) (unit 1)
+    (in_bom yes) (on_board yes)
+    (property "Reference" "U2" (id 0) (at 83.82 100.33 0))
+    (property "Value" "LOG114AIRGVR" (id 1) (at 50.8 101.6 0))
+    (property "Footprint" "Package_DFN_QFN:QFN-16-1EP_4x4mm_P0.65mm_EP2.15x2.15mm" (id 2) (at 64.77 92.71 0)
       (effects (font (size 1.27 1.27)) hide)
     )
-    (property "Datasheet" "https://www.ti.com/product/LOG114" (id 3) (at 77.47 96.52 0)
+    (property "Datasheet" "https://www.ti.com/product/LOG114" (id 3) (at 62.23 99.06 0)
       (effects (font (size 1.27 1.27)) hide)
     )

Commit message: update
Parts:
- removed U2: LOG114AIRGVR, Package_DFN_QFN:QFN-16-1EP_4x4mm_P0.65mm_EP2.15x2.15mm, symbol LOG114:LOG114AIRGVR
- renumbered U4 to U1, U3 to U2, U1 to U3
Connections:
- net amp1/+2.5V: now reaches U3.19 (OPD4)
- net amp2/+2.5V: now reaches U3.27 (OPD6)
- net amp1/I2: now reaches U3.48 (OPD4)
- net amp2/I2: now reaches U3.56 (OPD6)
Other:
- added sheet amp1 (amp.kicad_sch)
- added sheet amp2 (amp.kicad_sch)
- moved on the sheet: U1, U2, U3
